File: CANBusReaderBoard/CANBusReaderBoard.kicad_pcb (KiCad board)
At the start: 2 copper layers, 14 parts, among them J1 POWER -/+, J2 Terminate CAN, J3 CAN H/L, J4 CAN H/L

Commit message: printed board version
Parts:
- moved J1 7.87 mm to (144.8, 114.0)
Routing:
- net GNDREF: track 208.0 -> 194.7 mm
- net VCC: track 132.7 -> 120.4 mm
- added copper zone on B.Cu, net (none)
- added copper zone on F.Cu, net (none)
Other:
- board outline added: 52.6 x 78.4 mm
- board text added: "905-751-8626 defuria.alexander@gmail.com"
- board text added: "Designed By: Alexander De Furia"
- board text removed: "Designed By: Alexander De Furia 905-751-8626 defuria.alexander@gmail.com"
