File: RP2040/CANBusReaderBoard/CANBusReaderBoard.kicad_pcb (KiCad board)
At the start: 2 copper layers, 12.7 x 12.7 mm, 1 part, among them U1 RP2040

Commit message: .
Connections:
- U1 pad 52: unconnected-(U1-Pad52) -> /SPI_CLK
Changed lines of the file:
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@@
   (net 50 "unconnected-(U1-Pad50)")
   (net 51 "unconnected-(U1-Pad51)")
-  (net 52 "unconnected-(U1-Pad52)")
+  (net 52 "/SPI_CLK")
   (net 53 "unconnected-(U1-Pad53)")
   (net 54 "unconnected-(U1-Pad54)")
@@
       (net 51 "unconnected-(U1-Pad51)") (pinfunction "QSPI_SD3") (pintype "bidirectional"))
     (pad "52" smd roundrect (at -1 -3.435) (size 0.2 0.84) (layers "F.Cu" "F.Paste" "F.Mask") (roundrect_rratio 0.1)
-      (net 52 "unconnected-(U1-Pad52)") (pinfunction "QSPI_SCLK") (pintype "bidirectional"))
+      (net 52 "/SPI_CLK") (pinfunction "QSPI_SCLK") (pintype "bidirectional"))
     (pad "53" smd roundrect (at -1.4 -3.435) (size 0.2 0.84) (layers "F.Cu" "F.Paste" "F.Mask") (roundrect_rratio 0.1)
       (net 53 "unconnected-(U1-Pad53)") (pinfunction "QSPI_SD0") (pintype "bidirectional"))

Commit message: .
Parts:
- added C1: 100μF, Capacitor_THT:C_Axial_L3.8mm_D2.6mm_P7.50mm_Horizontal, F.Cu at (78.8, 144.8)
- added C2: 10μF, Capacitor_THT:C_Axial_L3.8mm_D2.6mm_P7.50mm_Horizontal, F.Cu at (112.8, 135.8)
- added C3: 15 pF, Capacitor_THT:C_Axial_L3.8mm_D2.6mm_P7.50mm_Horizontal, F.Cu at (119.7, 128.8)
- added C4: 15 pF, Capacitor_THT:C_Axial_L3.8mm_D2.6mm_P7.50mm_Horizontal, F.Cu at (78.8, 149.0)
- added C5: C 10u, Capacitor_THT:C_Axial_L3.8mm_D2.6mm_P7.50mm_Horizontal, F.Cu at (89.4, 149.0)
- added C6: C 10u, Capacitor_THT:C_Axial_L3.8mm_D2.6mm_P7.50mm_Horizontal, F.Cu at (89.4, 144.8)
- added J0: RJ45, Connector_RJ:RJ45_OST_PJ012-8P8CX_Vertical, F.Cu at (226.6, 105.9)
- added J1: RJ45, Connector_RJ:RJ45_OST_PJ012-8P8CX_Vertical, F.Cu at (226.6, 88.1)
- added J2: RJ45, Connector_RJ:RJ45_OST_PJ012-8P8CX_Vertical, F.Cu at (226.6, 70.4)
- added J4: Jack-DC, Connector_BarrelJack:BarrelJack_SwitchcraftConxall_RAPC10U_Horizontal, F.Cu at (168.7, 38.1)
- added J5: Terminate CAN, TerminalBlock_Phoenix:TerminalBlock_Phoenix_MKDS-3-2-5.08_1x02_P5.08mm_Horizontal, F.Cu at (157.5, 109.2)
- added R1: 10K, Resistor_THT:R_Axial_DIN0207_L6.3mm_D2.5mm_P10.16mm_Horizontal, F.Cu at (74.8, 165.7)
- added R2: 100, Resistor_THT:R_Axial_DIN0207_L6.3mm_D2.5mm_P10.16mm_Horizontal, F.Cu at (218.4, 96.5)
- added R3: 100, Resistor_THT:R_Axial_DIN0207_L6.3mm_D2.5mm_P10.16mm_Horizontal, F.Cu at (213.4, 106.7)
- added R4: 100, Resistor_THT:R_Axial_DIN0207_L6.3mm_D2.5mm_P10.16mm_Horizontal, F.Cu at (218.4, 78.7)
- added R5: 100, Resistor_THT:R_Axial_DIN0207_L6.3mm_D2.5mm_P10.16mm_Horizontal, F.Cu at (213.4, 88.9)
- added R6: 120, Resistor_THT:R_Axial_DIN0207_L6.3mm_D2.5mm_P10.16mm_Horizontal, F.Cu at (193.0, 121.9)
- added R7: 100, Resistor_THT:R_Axial_DIN0207_L6.3mm_D2.5mm_P10.16mm_Horizontal, F.Cu at (218.4, 61.0)
- added R8: 100, Resistor_THT:R_Axial_DIN0207_L6.3mm_D2.5mm_P10.16mm_Horizontal, F.Cu at (213.4, 71.1)
- added SW1: SW_DIP_x01, Button_Switch_THT:SW_DIP_SPSTx01_Slide_6.7x4.1mm_W7.62mm_P2.54mm_LowProfile, F.Cu at (88.1, 162.6)
- added U2: ATA00H18S-L, Converter_DCDC:Converter_DCDC_Artesyn_ATA_SMD, F.Cu at (223.5, 40.6)
- added U3: MCP2515-E/P, MCP2515-EP:MCP2515-E&slash_P, F.Cu at (156.2, 60.9)
- added U4: L78L05_SOT89, Package_TO_SOT_SMD:SOT-89-3, F.Cu at (188.0, 48.3)
- added U5: MCP2562-E-P, Package_DIP:DIP-8_W7.62mm, F.Cu at (156.2, 87.6)
- added Y1: Crystal 20Mhz, Crystal:Crystal_HC33-U_Vertical, F.Cu at (137.2, 76.2)
- U1: value RP2040 -> Pico; footprint RP2040:RP2040 -> MCU_RaspberryPi_and_Boards:RPi_Pico_StandOffs
- moved U1 48.3 mm to (185.4, 83.8)
Connections:
- U1 pad 1: unconnected-(U1-Pad1) -> MISO
- U1 pad 2: unconnected-(U1-Pad2) -> CS
- U1 pad 31: unconnected-(U1-Pad31) -> SENSOR 0
- U1 pad 32: unconnected-(U1-Pad32) -> SENSOR 1
- U1 pad 33: unconnected-(U1-Pad33) -> AGND
- U1 pad 34: unconnected-(U1-Pad34) -> SENSOR 2
- U1 pad 37: unconnected-(U1-Pad37) -> +3V3
- U1 pad 38: unconnected-(U1-Pad38) -> GND
- U1 pad 39: unconnected-(U1-Pad39) -> +5V
- U1 pad 4: unconnected-(U1-Pad4) -> SCLK
- U1 pad 5: unconnected-(U1-Pad5) -> MOSI
Routing:
- net SENSOR 0: track 0.00 -> 29.3 mm
- net SENSOR 2: track 0.00 -> 29.3 mm
- net SENSOR 1: track 0.00 -> 19.6 mm
- net GND1: track 0.00 -> 17.4 mm
- net Net-(J2-Pad4): track 0.00 -> 12.5 mm
- net Net-(J1-Pad4): track 0.00 -> 12.5 mm
- net Net-(J0-Pad4): track 0.00 -> 12.5 mm
Other:
- board outline removed

Commit message: ready for wiring
Parts:
- removed J0: RJ45, Connector_RJ:RJ45_OST_PJ012-8P8CX_Vertical
- added D1: Inolux_IN-PI554FCH, LED_SMD:LED_Inolux_IN-PI554FCH_PLCC4_5.0x5.0mm_P3.2mm, F.Cu at (239.0, 143.5)
- added D2: Inolux_IN-PI554FCH, LED_SMD:LED_Inolux_IN-PI554FCH_PLCC4_5.0x5.0mm_P3.2mm, F.Cu at (247.0, 143.5)
- added D3: Inolux_IN-PI554FCH, LED_SMD:LED_Inolux_IN-PI554FCH_PLCC4_5.0x5.0mm_P3.2mm, F.Cu at (231.1, 143.5)
- added D4: Inolux_IN-PI554FCH, LED_SMD:LED_Inolux_IN-PI554FCH_PLCC4_5.0x5.0mm_P3.2mm, F.Cu at (231.1, 150.1)
- added D5: Inolux_IN-PI554FCH, LED_SMD:LED_Inolux_IN-PI554FCH_PLCC4_5.0x5.0mm_P3.2mm, F.Cu at (239.0, 150.1)
- added R10: 500, Resistor_THT:R_Axial_DIN0207_L6.3mm_D2.5mm_P10.16mm_Horizontal, F.Cu at (184.2, 135.8)
- added R11: 500, Resistor_THT:R_Axial_DIN0207_L6.3mm_D2.5mm_P10.16mm_Horizontal, F.Cu at (184.2, 131.8)
- added R12: 500, Resistor_THT:R_Axial_DIN0207_L6.3mm_D2.5mm_P10.16mm_Horizontal, F.Cu at (184.2, 127.7)
- added R9: 500, Resistor_THT:R_Axial_DIN0207_L6.3mm_D2.5mm_P10.16mm_Horizontal, F.Cu at (179.6, 155.2)
- J1: value RJ45 -> Conn_01x10_Female; footprint Connector_RJ:RJ45_OST_PJ012-8P8CX_Vertical -> Connector_PinHeader_2.54mm:PinHeader_1x10_P2.54mm_Vertical
- J2: value RJ45 -> 3xRJ45V; footprint Connector_RJ:RJ45_OST_PJ012-8P8CX_Vertical -> 3xRJ45V:3xRJ45V
- moved J1 57.9 mm to (169.7, 77.5), turned to 0 degrees
- moved C2 54.4 mm to (165.4, 122.0)
- moved C3 54.4 mm to (172.3, 115.0)
- moved SW1 54.4 mm to (140.7, 148.7)
- moved C1 54.4 mm to (131.4, 131.0)
- moved C4 54.4 mm to (131.4, 135.1)
- moved C5 54.4 mm to (142.0, 135.1)
- moved C6 54.4 mm to (142.0, 131.0)
- moved R1 54.4 mm to (127.4, 151.9)
- moved J2 36.3 mm to (230.4, 106.5)
Connections:
- J1 pad 1: +24V -> Net-(J1-Pad1)
- J1 pad 2: unconnected-(J1-Pad2) -> Net-(J1-Pad2)
- J1 pad 3: unconnected-(J1-Pad3) -> Net-(J1-Pad3)
- J1 pad 5: unconnected-(J1-Pad5) -> Net-(J1-Pad5)
- J1 pad 6: unconnected-(J1-Pad6) -> Net-(J1-Pad6)
- J1 pad 7: unconnected-(J1-Pad7) -> Net-(J1-Pad7)
- J1 pad 8: GND1 -> Net-(J1-Pad8)
- R2 pad 2: Net-(J0-Pad4) -> SENSOR 0 (24V)
- R3 pad 1: Net-(J0-Pad4) -> SENSOR 0 (24V)
- R4 pad 2: Net-(J1-Pad4) -> SENSOR 1 (24V)
- R5 pad 1: Net-(J1-Pad4) -> SENSOR 1 (24V)
- R7 pad 2: Net-(J2-Pad4) -> SENSOR 2 (24V)
- R8 pad 1: Net-(J2-Pad4) -> SENSOR 2 (24V)
- U1 pad 10: unconnected-(U1-Pad10) -> Net-(J1-Pad3)
- U1 pad 11: unconnected-(U1-Pad11) -> Net-(J1-Pad4)
- U1 pad 12: unconnected-(U1-Pad12) -> Net-(J1-Pad5)
- U1 pad 13: unconnected-(U1-Pad13) -> Net-(J1-Pad6)
- U1 pad 14: unconnected-(U1-Pad14) -> Net-(J1-Pad7)
- U1 pad 15: unconnected-(U1-Pad15) -> Net-(J1-Pad8)
- U1 pad 16: unconnected-(U1-Pad16) -> Net-(J1-Pad9)
- U1 pad 17: unconnected-(U1-Pad17) -> Net-(J1-Pad10)
- U1 pad 26: unconnected-(U1-Pad26) -> LED1
- U1 pad 27: unconnected-(U1-Pad27) -> LED2
- U1 pad 8: unconnected-(U1-Pad8) -> Net-(J1-Pad1)
- U1 pad 9: unconnected-(U1-Pad9) -> Net-(J1-Pad2)
Routing:
- net GND1: track 17.4 -> 0.00 mm
- net Net-(J2-Pad4): track 12.5 -> 0.00 mm
- net Net-(J1-Pad4): track 12.5 -> 0.00 mm
- net Net-(J0-Pad4): track 12.5 -> 0.00 mm
- net SENSOR 2 (24V): track 0.00 -> 6.10 mm
- net SENSOR 1 (24V): track 0.00 -> 6.10 mm
- net SENSOR 0 (24V): track 0.00 -> 6.10 mm

Commit message: Finished footprints and started initial track laying
Parts:
- removed U2: ATA00H18S-L, Converter_DCDC:Converter_DCDC_Artesyn_ATA_SMD
- added PS1: ITQ4805SA-H, Converter_DCDC:Converter_DCDC_XP_POWER-ITQxxxxS-H_THT, F.Cu at (167.1, 45.1)
- C1: footprint Capacitor_THT:C_Axial_L3.8mm_D2.6mm_P7.50mm_Horizontal -> Capacitor_THT:CP_Radial_D5.0mm_P2.00mm
- C2, C3, C4, C5, C6: footprint Capacitor_THT:C_Axial_L3.8mm_D2.6mm_P7.50mm_Horizontal -> Capacitor_SMD:C_1206_3216Metric_Pad1.33x1.80mm_HandSolder
- J4: footprint Connector_BarrelJack:BarrelJack_SwitchcraftConxall_RAPC10U_Horizontal -> Connector_BarrelJack:BarrelJack_CUI_PJ-063AH_Horizontal
- R1, R6: footprint Resistor_THT:R_Axial_DIN0207_L6.3mm_D2.5mm_P10.16mm_Horizontal -> Resistor_SMD:R_1206_3216Metric_Pad1.30x1.75mm_HandSolder
- R10, R11, R12, R9: value 500 -> 499; footprint Resistor_THT:R_Axial_DIN0207_L6.3mm_D2.5mm_P10.16mm_Horizontal -> Resistor_SMD:R_1206_3216Metric_Pad1.30x1.75mm_HandSolder
- R2, R4, R7: value 100 -> 3.3; footprint Resistor_THT:R_Axial_DIN0207_L6.3mm_D2.5mm_P10.16mm_Horizontal -> Resistor_SMD:R_1206_3216Metric_Pad1.30x1.75mm_HandSolder
- R3, R5, R8: value 100 -> 6.8; footprint Resistor_THT:R_Axial_DIN0207_L6.3mm_D2.5mm_P10.16mm_Horizontal -> Resistor_SMD:R_1206_3216Metric_Pad1.30x1.75mm_HandSolder
- U4: value L78L05_SOT89 -> NCV5501DT50RKG; footprint Package_TO_SOT_SMD:SOT-89-3 -> Package_TO_SOT_SMD:TO-252-2
- Y1: footprint Crystal:Crystal_HC33-U_Vertical -> Crystal:Crystal_HC49-4H_Vertical
- moved D2 168.6 mm to (107.4, 48.8)
- moved D4 153.6 mm to (115.3, 49.0)
- moved R10 120.0 mm to (101.6, 48.8), turned to -90 degrees
- moved D1 116.4 mm to (154.7, 63.2), turned to 180 degrees
- moved D5 111.9 mm to (154.7, 76.5), turned to 180 degrees
- moved D3 106.1 mm to (154.7, 69.8), turned to 180 degrees
- moved R11 105.0 mm to (121.9, 47.2), turned to 180 degrees
- moved R9 99.3 mm to (155.4, 58.9)
- moved R6 96.3 mm to (100.3, 95.8), turned to 90 degrees
- moved C5 85.0 mm to (142.2, 50.1), turned to 90 degrees
- moved C1 84.9 mm to (169.6, 55.1), turned to 180 degrees
- moved C6 81.6 mm to (131.1, 50.1), turned to 90 degrees
- moved C4 74.2 mm to (118.7, 62.1), turned to -90 degrees
- moved C3 71.3 mm to (118.6, 68.1), turned to -90 degrees
- moved R1 70.6 mm to (101.1, 86.4), turned to -90 degrees
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Connections:
- D1 pad 1: GND -> GNDREF
- D2 pad 1: GND -> GNDREF
- D3 pad 1: GND -> GNDREF
- D4 pad 1: GND -> GNDREF
- D5 pad 1: GND -> GNDREF
- U1 pad 18: unconnected-(U1-Pad18) -> GND
- U1 pad 23: unconnected-(U1-Pad23) -> GND
- U1 pad 3: unconnected-(U1-Pad3) -> GND
- U1 pad 39: +5V -> unconnected-(U1-Pad39)
- U1 pad 40: unconnected-(U1-Pad40) -> +5V
- U3 pad 13: SPICLK -> SCLK
- U3 pad 16: CS0 -> CS
- U3 pad 18: GND -> +3V3
- U3 pad 9: +3V3 -> GND
- U5 pad 2: +3V3 -> GND
- U5 pad 3: GND -> +3V3
Routing:
- net GND: track 0.00 -> 85.1 mm, vias 0 -> 1
- net MOSI: track 0.00 -> 54.7 mm
- net LED1: track 0.00 -> 52.0 mm
- net +12V: track 0.00 -> 46.3 mm
- net SCLK: track 0.00 -> 43.9 mm
- net CS: track 0.00 -> 39.5 mm
- net MISO: track 0.00 -> 36.7 mm
- net CANH: track 0.00 -> 31.4 mm
- net SENSOR 2 (24V): track 6.10 -> 29.8 mm
- net CANL: track 0.00 -> 20.7 mm
- net +3V3: track 0.00 -> 19.2 mm
- net SENSOR 1 (24V): track 6.10 -> 22.8 mm
- net TX: track 0.00 -> 15.3 mm
- net Net-(C3-Pad2): track 0.00 -> 11.6 mm
- net SENSOR 0 (24V): track 6.10 -> 17.4 mm
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
Commit message: printed
Parts:
- removed J1: Conn_01x10_Female, Connector_PinHeader_2.54mm:PinHeader_1x10_P2.54mm_Vertical
- removed R10, R12: 499, Resistor_SMD:R_1206_3216Metric_Pad1.30x1.75mm_HandSolder
- added G***: LOGO, LOGO, F.Cu at (156.5, 61.7)
- added REF**: MountingHole_2.5mm_Pad, MountingHole:MountingHole_2.5mm_Pad, F.Cu at (108.3, 107.1)
- added REF**: MountingHole_2.5mm_Pad, MountingHole:MountingHole_2.5mm_Pad, F.Cu at (148.6, 106.0)
- added REF**: MountingHole_2.5mm_Pad, MountingHole:MountingHole_2.5mm_Pad, F.Cu at (131.5, 48.5)
- added REF**: MountingHole_2.5mm_Pad, MountingHole:MountingHole_2.5mm_Pad, F.Cu at (171.0, 48.6)
- added REF**: MountingHole_2.5mm_Pad, MountingHole:MountingHole_2.5mm_Pad, F.Cu at (119.9, 81.3)
- added REF**: MountingHole_2.5mm_Pad, MountingHole:MountingHole_2.5mm_Pad, F.Cu at (148.6, 66.7)
- C5, C6: value C 10u -> 10μF
- R6: value 120 -> 120k
- moved R11 45.2 mm to (167.1, 48.8), turned to -90 degrees
- moved D4 39.1 mm to (154.4, 48.8)
- moved J4 38.6 mm to (117.3, 52.3), turned to -90 degrees
- moved C2 33.1 mm to (148.6, 61.0), turned to 90 degrees
- moved D2 31.8 mm to (139.2, 48.8)
- moved D5 28.6 mm to (162.1, 48.8), turned to 0 degrees
- moved D3 22.5 mm to (146.8, 48.8), turned to 0 degrees
- moved C1 22.3 mm to (147.3, 53.9), turned to -90 degrees
- moved C5 22.2 mm to (120.1, 50.8)
- moved R9 21.9 mm to (134.0, 54.4), turned to 90 degrees
- moved D1 17.6 mm to (139.2, 54.9), turned to 0 degrees
- moved R7 16.9 mm to (148.6, 72.9), turned to -90 degrees
- moved PS1 16.5 mm to (154.3, 55.5)
- moved R8 14.5 mm to (148.6, 78.3), turned to -90 degrees
- moved R4 14.2 mm to (148.6, 83.7), turned to -90 degrees
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Connections:
- C1 pad 2: Net-(C1-Pad2) -> GNDREF
- C2 pad 2: GND1 -> AGND
- C3 pad 1: GND -> GND3
- C4 pad 1: GND -> GND3
- D2 pad 2: Net-(D2-Pad2) -> Net-(D1-Pad4)
- D2 pad 4: Net-(D2-Pad4) -> Net-(D3-Pad2)
- D3 pad 2: Net-(D1-Pad4) -> Net-(D3-Pad2)
- D3 pad 4: Net-(D3-Pad4) -> Net-(D4-Pad2)
- D4 pad 2: Net-(D2-Pad4) -> Net-(D4-Pad2)
- D5 pad 2: Net-(D3-Pad4) -> Net-(D4-Pad4)
- J2 pad A8: GND1 -> AGND
- J2 pad B8: GND1 -> AGND
- J2 pad C8: GND1 -> AGND
- J4 pad 2: Net-(C1-Pad2) -> GNDREF
- PS1 pad 1: Net-(C1-Pad2) -> GNDREF
- PS1 pad 7: GND1 -> AGND
- R11 pad 1: Net-(D4-Pad4) -> Net-(D5-Pad4)
- R11 pad 2: GND -> GNDREF
- R2 pad 1: GND1 -> AGND
- R4 pad 1: GND1 -> AGND
- R7 pad 1: GND1 -> AGND
- U1 pad 10: Net-(J1-Pad3) -> unconnected-(U1-Pad10)
- U1 pad 11: Net-(J1-Pad4) -> unconnected-(U1-Pad11)
- U1 pad 12: Net-(J1-Pad5) -> unconnected-(U1-Pad12)
- U1 pad 13: Net-(J1-Pad6) -> unconnected-(U1-Pad13)
- U1 pad 14: Net-(J1-Pad7) -> unconnected-(U1-Pad14)
- U1 pad 15: Net-(J1-Pad8) -> unconnected-(U1-Pad15)
- U1 pad 16: Net-(J1-Pad9) -> unconnected-(U1-Pad16)
- U1 pad 17: Net-(J1-Pad10) -> unconnected-(U1-Pad17)
- U1 pad 18: GND -> GND3
- U1 pad 26: LED1 -> LED2
- U1 pad 27: LED2 -> LED1
- U1 pad 3: GND -> GND2
- U1 pad 38: GND -> GNDREF
- U1 pad 8: Net-(J1-Pad1) -> unconnected-(U1-Pad8)
- U1 pad 9: Net-(J1-Pad2) -> unconnected-(U1-Pad9)
- U3 pad 9: GND -> GND3
- U5 pad 2: GND -> GND3
Routing:
- net GNDREF: track 7.63 -> 177.9 mm
- net AGND: track 0.00 -> 132.5 mm, vias 0 -> 3
- net GND: track 85.1 -> 0.00 mm, vias 1 -> 0
- net +3V3: track 19.2 -> 98.9 mm, vias 0 -> 1
- net GND3: track 0.00 -> 75.3 mm
- net +24V: track 9.65 -> 73.8 mm
- net +5V: track 0.00 -> 53.2 mm
- net SENSOR 2 (24V): track 29.8 -> 11.6 mm
- net SENSOR 2: track 22.5 -> 8.51 mm
- net SENSOR 1: track 25.4 -> 12.2 mm
- net SENSOR 1 (24V): track 22.8 -> 11.3 mm
- net Net-(C1-Pad2): track 10.2 -> 0.00 mm
- net SENSOR 0: track 31.2 -> 21.4 mm
- net GND1: track 9.65 -> 0.00 mm
- net MOSI: track 54.7 -> 47.4 mm
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- added copper zone on B.Cu, net (none)
- added copper zone on F.Cu, net (none)
Other:
- board outline added: 70 x 66.4 mm
- board text added: "10V to 3.3V Voltage Divider"
- board text added: "12V"
- board text added: "15.24X 37.04Y"
- board text added: "2.5mm"
- board text added: "20MHz"
- board text added: "26.85X 4.19Y"
- board text added: "3.65X 62.79Y"
- board text added: "43.94X 22.37Y"
- board text added: "43.94X 61.69Y"
- board text added: "5V"
- board text added: "66.35X 4.29Y"
- board text added: "Alexander DeFuria FRC CANBusReaderBoard 905-751-8626 defuria.alexander@gmail.com"
- board text added: "Balluff Sensors operate at 24V. Pin 1: Power (+24V) Pin 5: Analog Data (0..10V) Pin 8: GND (-)"
- board text added: "Board Dimensions Width: 70mm Height: 66.5mm"
- board text added: "DO NOT POWER BOARD BY BOTH USB AND 12V POWER"
- board text added: "Flip switch to terminate canbus."
- board text added: "H / L"
- board text added: "JLCJLCJLCJLC"
- board text added: "Jack A GP 26"
- board text added: "Jack B GP 27"
- board text added: "Jack C GP 28"
- board text added: "MCP2515-E/P"
- board text added: "MCP2562-E-P"
- board text added: "MCP2562-FD"
- board text added: "MISO GP0 CS GP1 SCLK GP2 MOSI GP3"
- board text added: "Mounting holes are 2.5mm diameter Pad is 5mm diameter LEDs are Inolux IN-PI554FCH Digital LEDs"
- board text added: "OFF"
- board text added: "ON"
- board text added: "Raspberry Pi Pico Sensors GP26-28 Lights GP20-21"
- board text added: "Raspberry Pi Pico Sensors GP26-28 Lights GP21"
- board text added: "V2.1"
- board text added: "Voltage divider from 0..10V to 0..3.3V"
- board text added: "X0Y0(mm)"
- board text added: "You're welcome for the excessive docs ;)"
