File: RP2040/CANBusReaderBoard/CANBusReaderBoard.kicad_sch (KiCad schematic)
At the start: 34 parts, among them J1 Conn_01x10_Female, J2 3xRJ45V, J4 Jack-DC, J5 Terminate CAN, SW1 SW_DIP_x01, U1 Pico, U2 ATA00H18S-L, U3 MCP2515-E{slash}P, U4 L78L05_SOT89, U5 MCP2562-E-P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

Commit message: Finished footprints and started initial track laying
Parts:
- removed U2: ATA00H18S-L, Converter_DCDC:Converter_DCDC_Artesyn_ATA_SMD, symbol Converter_DCDC:ATA00H18S-L
- added PS1: ITQ4805SA-H, Converter_DCDC:Converter_DCDC_XP_POWER-ITQxxxxS-H_THT, symbol Converter_DCDC:ITQ4805SA-H
- C1: footprint Capacitor_THT:C_Axial_L3.8mm_D2.6mm_P7.50mm_Horizontal -> Capacitor_THT:CP_Radial_D5.0mm_P2.00mm
- C2, C3, C4, C5, C6: footprint Capacitor_THT:C_Axial_L3.8mm_D2.6mm_P7.50mm_Horizontal -> Capacitor_SMD:C_1206_3216Metric_Pad1.33x1.80mm_HandSolder
- J4: footprint Connector_BarrelJack:BarrelJack_SwitchcraftConxall_RAPC10U_Horizontal -> Connector_BarrelJack:BarrelJack_CUI_PJ-063AH_Horizontal
- R1, R6: footprint Resistor_THT:R_Axial_DIN0207_L6.3mm_D2.5mm_P10.16mm_Horizontal -> Resistor_SMD:R_1206_3216Metric_Pad1.30x1.75mm_HandSolder
- R10, R11, R12, R9: value 500 -> 499; footprint Resistor_THT:R_Axial_DIN0207_L6.3mm_D2.5mm_P10.16mm_Horizontal -> Resistor_SMD:R_1206_3216Metric_Pad1.30x1.75mm_HandSolder
- R2, R4, R7: value 100 -> 3.3; footprint Resistor_THT:R_Axial_DIN0207_L6.3mm_D2.5mm_P10.16mm_Horizontal -> Resistor_SMD:R_1206_3216Metric_Pad1.30x1.75mm_HandSolder
- R3, R5, R8: value 100 -> 6.8; footprint Resistor_THT:R_Axial_DIN0207_L6.3mm_D2.5mm_P10.16mm_Horizontal -> Resistor_SMD:R_1206_3216Metric_Pad1.30x1.75mm_HandSolder
- U4: value L78L05_SOT89 -> NCV5501DT50RKG; footprint Package_TO_SOT_SMD:SOT-89-3 -> Package_TO_SOT_SMD:TO-252-2
- Y1: footprint Crystal:Crystal_HC33-U_Vertical -> Crystal:Crystal_HC49-4H_Vertical
Connections:
- net CS0 is gone; now on net CS: U3.16 (*CS)
- net SPICLK is gone; now on net SCLK: U3.13 (SCK)
- net +12V: now also PS1.2 (+Vin)
- net +24V: now also PS1.6 (+Vout)
- net +3V3: now also U3.18 (VDD), U5.3 (VDD); no longer U3.9 (VSS), U5.2 (VSS)
- net +5V: now also U1.40 (VBUS); no longer U1.39 (VSYS)
- net GND: now also U1.18 (GND), U1.23 (GND), U1.3 (GND), U3.9 (VSS), U5.2 (VSS); no longer D1.1 (VSS), D2.1 (VSS), D3.1 (VSS), D4.1 (VSS), D5.1 (VSS), U3.18 (VDD), U5.3 (VDD)
- net GND1: now also PS1.7 (-Vout)
- net GNDREF: now also D1.1 (VSS), D2.1 (VSS), D3.1 (VSS), D4.1 (VSS), D5.1 (VSS)
- net at C1.2, J4.2: now also PS1.1 (-Vin)
Other:
- note added: "DC Regulator to 5V"
- note removed: "DC Regulator to 3.3V"
- moved on the sheet: C2, R11, R12

Commit message: printed
Parts:
- removed J1: Conn_01x10_Female, Connector_PinHeader_2.54mm:PinHeader_1x10_P2.54mm_Vertical, symbol Connector:Conn_01x10_Female
- removed R10, R12: 499, Resistor_SMD:R_1206_3216Metric_Pad1.30x1.75mm_HandSolder, symbol Device:R
- C5, C6: value C 10u -> 10μF
- R6: value 120 -> 120k
- renumbered D3 to D2, D5 to D3, D2 to D4, D4 to D5
Connections:
- net AGND is gone; now on net GND1: U1.33 (AGND)
- net GND: no longer C3.1, C4.1, R11.2, U1.18 (GND), U1.3 (GND), U1.38 (GND), U3.9 (VSS), U5.2 (VSS)
- net GNDREF: now also C1.2, J4.2, PS1.1 (-Vin), R11.2, U1.38 (GND)
- net LED1: now also U1.27 (GPIO21); no longer U1.26 (GPIO20)
- net LED2: now also U1.26 (GPIO20); no longer U1.27 (GPIO21)
- net at D3.4 (DO): now also D4.2 (DIN)
- new net GND2: U1.3 (GND)
- new net GND3: C3.1, C4.1, U1.18 (GND), U3.9 (VSS), U5.2 (VSS)
Other:
- moved on the sheet: D1, D2, D3, D4, D5, R11, R9
